File: broampexg.kicad_pcb (KiCad board)
At the start: 2 copper layers, 36.5 x 48 mm, 26 parts, among them J1 BioAmp Output, J2 BioAmp Input, U1 Amp

Commit message: fonts and stuff yay
Other:
- board text added: "easter egg"
- board text added: "not-willem"
