File: broampexg.kicad_pcb (KiCad board)
At the start: 2 copper layers, 36.5 x 48 mm, 26 parts, among them J1 BioAmp Output, J2 BioAmp Input, U1 Amp

Commit message: named the caps and res
doorman doorstop doormouse doorframe doorknob doordash
Other:
- board text added: "R0r"
- board text added: "R1M"
- board text added: "R1k"
- board text added: "R220k"
- board text added: "R22k"
- board text added: "TL074HIPWR"
- board text added: "c100nF"
- board text added: "c10uF"
- board text added: "c1nF"
- board text added: "c47uF"
