File: broampexg.kicad_pcb (KiCad board)
At the start: 2 copper layers, 36.5 x 48 mm, 26 parts, among them J1 BioAmp Output, J2 BioAmp Input, U1 Amp

Commit message: added source qr on pcb
hooray!
Parts:
- added ?: LOGO, component:sourceqr, F.Cu at (73.2, 83.0)
Other:
- board text added: "source"

Commit message: ooh wah doo wap doopity doo
wow
Other:
- board text added: "Original design: Upside Down Labs BioAmp EXG Pill, MAR 2023. Modified by Willem van Hulst, June 2026. More info at source, scan the qr code at the front of the board"
